File: pcb/connectors.kicad_sch (KiCad schematic)
At the start: 3 parts, among them X501 PH-00650, X502 S4B-PH-SM4-K-TB(LF)(SN), X503 USB3.1C16PFSMT

Commit message: make it work
Parts:
- removed X501: PH-00650, HDR-SMD_40P-P2.54-V-M-R2-C20-S7.8-EH, symbol eduboardv2:PH-00650
- removed X502: S4B-PH-SM4-K-TB(LF)(SN), CONN-SMD_S4B-PH-SM4-K-TB-LF-SN, symbol eduboardv2:S4B-PH-SM4-K-TB(LF)(SN)
Connections:
- removed net GND: X503.0, X503.A1 (GND), X503.A12 (GND)
- no-connect marks 0 -> 6
Changed lines of the file:
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@@
   (junction (at 162.56 74.93) (diameter 0) (color 0 0 0 0)
   )
+  (no_connect (at 175.26 100.33))
+  (no_connect (at 152.4 92.71))
+  (no_connect (at 152.4 100.33))
+  (no_connect (at 175.26 102.87))
+  (no_connect (at 175.26 92.71))
+  (no_connect (at 175.26 90.17))
   (wire (pts (xy 137.16 97.79) (xy 152.4 97.79))
     (stroke (width 0) (type default) (color 0 0 0 0))
@@
     (effects (font (size 1.27 1.27)) (justify left bottom))
   )
-  (symbol (lib_id "power:GND") (at 175.26 82.55 0) (unit 1)
+  (symbol (lib_id "eduboardv2:GND") (at 175.26 82.55 0) (unit 1)
     (in_bom yes) (on_board yes) (fields_autoplaced)
     (property "Reference" "#PWR0503" (id 0) (at 175.26 88.9 0)
@@
     (pin "1")
   )
-  (symbol (lib_id "eduboardv2:PH-00650") (at 78.74 81.28 0) (unit 1)
-    (in_bom yes) (on_board yes) (fields_autoplaced)
-    (property "Reference" "X501" (id 0) (at 78.74 49.53 0))
-    (property "Value" "PH-00650" (id 1) (at 78.74 52.07 0))
-    (property "Footprint" "HDR-SMD_40P-P2.54-V-M-R2-C20-S7.8-EH" (id 2) (at 78.74 113.03 0)
-      (effects (font (size 1.27 1.27)) hide)
-    )
-    (property "Datasheet" "" (id 3) (at 78.74 81.28 0)
-      (effects (font (size 1.27 1.27)) hide)
-    )
-    (property "Manufacturer" "Liansheng(连盛)" (id 4) (at 78.74 118.11 0)
-      (effects (font (size 1.27 1.27)) hide)
-    )
-    (property "LCSC Part" "C2685175" (id 5) (at 78.74 120.65 0)
-      (effects (font (size 1.27 1.27)) hide)
-    )
-    (property "JLC Part" "Extended Part" (id 6) (at 78.74 123.19 0)
-      (effects (font (size 1.27 1.27)) hide)
-    )
-    (property "MPN" "PH-00650" (id 7) (at 78.74 110.49 0)
-      (effects (font (size 1.27 1.27)) hide)
-    )
-    (pin "1")
-    (pin "10")
-    (pin "11")
-    (pin "12")
-    (pin "13")
-    (pin "14")
-    (pin "15")
-    (pin "16")
-    (pin "17")
-    (pin "18")
-    (pin "19")
-    (pin "2")
-    (pin "20")
-    (pin "21")
-    (pin "22")
-    (pin "23")
-    (pin "24")
-    (pin "25")
-    (pin "26")
-    (pin "27")
-    (pin "28")
-    (pin "29")
-    (pin "3")
-    (pin "30")
-    (pin "31")
-    (pin "32")
-    (pin "33")
-    (pin "34")
-    (pin "35")
-    (pin "36")
-    (pin "37")
-    (pin "38")
-    (pin "39")
-    (pin "4")
-    (pin "40")
-    (pin "5")
-    (pin "6")
-    (pin "7")
-    (pin "8")
-    (pin "9")
-  )
-  (symbol (lib_id "power:GND") (at 175.26 110.49 0) (unit 1)
+  (symbol (lib_name "GND_3") (lib_id "eduboardv2:GND") (at 175.26 110.49 0) (unit 1)
     (in_bom yes) (on_board yes) (fields_autoplaced)
     (property "Reference" "#PWR0504" (id 0) (at 175.26 116.84 0)
@@
     (pin "1")
   )
-  (symbol (lib_id "power:GND") (at 162.56 115.57 0) (unit 1)
+  (symbol (lib_name "GND_2") (lib_id "eduboardv2:GND") (at 162.56 115.57 0) (unit 1)
     (in_bom yes) (on_board yes) (fields_autoplaced)
     (property "Reference" "#PWR0502" (id 0) (at 162.56 121.92 0)
@@
     (pin "1")
   )
-  (symbol (lib_id "power:GND") (at 157.48 72.39 0) (unit 1)
+  (symbol (lib_name "GND_1") (lib_id "eduboardv2:GND") (at 157.48 72.39 0) (unit 1)
     (in_bom yes) (on_board yes) (fields_autoplaced)
     (property "Reference" "#PWR0501" (id 0) (at 157.48 78.74 0)
@@
     (pin "1")
   )
-  (symbol (lib_id "eduboardv2:S4B-PH-SM4-K-TB(LF)(SN)") (at 156.21 38.1 0) (unit 1)
-    (in_bom yes) (on_board yes) (fields_autoplaced)
-    (property "Reference" "X502" (id 0) (at 165.1 38.0999 0)
-      (effects (font (size 1.27 1.27)) (justify left))
-    )
-    (property "Value" "S4B-PH-SM4-K-TB(LF)(SN)" (id 1) (at 165.1 40.6399 0)
-      (effects (font (size 1.27 1.27)) (justify left))
-    )
-    (property "Footprint" "CONN-SMD_S4B-PH-SM4-K-TB-LF-SN" (id 2) (at 156.21 55.88 0)
-      (effects (font (size 1.27 1.27)) hide)
-    )
-    (property "Datasheet" "https://lcsc.com/product-detail/Others_JST-Sales-America_S4B-PH-SM4-K-TB-LF-SN_JST-Sales-America-S4B-PH-SM4-K-TB-LF-SN_C265332.html" (id 3) (at 156.21 60.96 0)
-      (effects (font (size 1.27 1.27)) hide)
-    )
-    (property "Manufacturer" "JST Sales America" (id 4) (at 156.21 63.5 0)
-      (effects (font (size 1.27 1.27)) hide)
-    )
-    (property "LCSC Part" "C265332" (id 5) (at 156.21 66.04 0)
-      (effects (font (size 1.27 1.27)) hide)
-    )
-    (property "JLC Part" "Extended Part" (id 6) (at 156.21 68.58 0)
-      (effects (font (size 1.27 1.27)) hide)
-    )
-    (property "MPN" "S4B-PH-SM4-K-TB(LF)(SN)" (id 7) (at 156.21 53.34 0)
-      (effects (font (size 1.27 1.27)) hide)
-    )
-    (pin "1")
-    (pin "2")
-    (pin "3")
-    (pin "4")
-    (pin "5")
-    (pin "6")
-  )
   (symbol (lib_id "eduboardv2:USB3.1C16PFSMT") (at 163.83 96.52 0) (unit 1)
