File: pcb/display_ui.kicad_sch (KiCad schematic)
At the start: 68 parts, among them SW401 K2-1102SP-C4SC-04, SW402 K2-1102SP-C4SC-04, SW403 K2-1102SP-C4SC-04, SW404 K2-1102SP-C4SC-04, T401 AO3400A, T402 AO3400A, T403 AO3400A, T404 AO3400A, T405 AO3400A, X401 ER-TFT035-6

Commit message: make it work
Connections:
- removed net +3.3V: BUZZER401.1 (+), C409.2, C410.2, C411.2, D409.3 (A), D411.1 (K), R401.2, R404.3, R408.2, R411.3, R415.3, R416.2, R420.2, R428.1, R430.1, R433.1, R435.2, X401.13 (DOTCLK), X401.35 (RD), X401.40 (VDDI), X401.41 (VDDI), X401.42 (VCI)
- removed net GND: C401.1, C402.1, C403.1, C404.1, C405.1, C406.1, C407.1, C408.1, C409.1, C410.1, C411.1, D401.2 (C), D402.2 (C), D403.2 (C), D404.2 (C), D405.2 (C), D406.2 (C), D407.2 (C), D408.2 (C), D410.3 (VSS), R402.1, R404.1, R409.1, R411.1, R415.1, R417.1, R421.1, R429.2, R431.2, R434.2, T401.2 (S), T402.2 (S), T403.2 (S), T404.2 (S), T405.2 (S), X401.11 (VSYNC), X401.12 (HSYNC), X401.14 (DE), X401.15 (DB17), X401.16 (DB16), X401.17 (DB15), X401.18 (DB14), X401.19 (DB13), X401.20 (DB12), X401.21 (DB11), X401.22 (DB10), X401.23 (DB9), X401.24 (DB8), X401.25 (DB7), X401.26 (DB6), X401.27 (DB5), X401.28 (DB4), X401.29 (DB3), X401.30 (DB2), X401.31 (DB1), X401.32 (DB0), X401.43 (GND), X401.48 (GND), X401.49 (GND), X401.50 (GND)
- new net: C409.1, C410.1, C411.1
- new net: C409.2, C410.2, C411.2
- new net: R428.1, R430.1, R433.1
- new net: BUZZER401.1 (+), D411.1 (K)
- new net: X401.11 (VSYNC), X401.12 (HSYNC)
- new net: X401.14 (DE), X401.15 (DB17), X401.16 (DB16), X401.17 (DB15), X401.18 (DB14), X401.19 (DB13), X401.20 (DB12), X401.21 (DB11), X401.22 (DB10), X401.23 (DB9), X401.24 (DB8), X401.25 (DB7), X401.26 (DB6), X401.27 (DB5), X401.28 (DB4), X401.29 (DB3), X401.30 (DB2), X401.31 (DB1), X401.32 (DB0)
- new net: X401.40 (VDDI), X401.41 (VDDI), X401.42 (VCI)
- new net: X401.48 (GND), X401.49 (GND), X401.50 (GND)
- new net: R429.2, R431.2, R434.2
- no-connect marks 0 -> 18
