File: pcb/power.kicad_sch (KiCad schematic)
At the start: 35 parts, among them IC301 XL1509-5.0E1, IC302 SY8113BADC, X301 KF2EDGR-3.81-3P, X302 USB3.1C16PFSMT, X303 CH340G, Y301 X322512MSB4SI

Commit message: make it work
Parts:
- added SW301: 1FS1T1B9M2RES-5, SW-TH_1FS1T1B9M2RES-5, symbol eduboardv2:1FS1T1B9M2RES-5
Connections:
- net +3.3V: no longer names the net of C308.2, C310.2, C312.1, C314.1, C316.1, D305.1 (A), L301.2, R305.2
- net +5V: no longer names the net of C307.2, IC302.5 (IN), R303.2
- net +5V: no longer D302.1 (K), D303.1 (K)
- net +5V_EXT: no longer names the net of C309.1, C311.1, C313.2, C315.1, IC301.3 (FB), L302.2
- net +5V_EXT: no longer D303.2 (A)
- removed net GND: C301.2, C302.1, C303.1, C304.1, C305.1, C307.1, C309.2, C310.1, C311.2, C312.2, C313.1, C314.2, C315.2, C316.2, D301.2 (A), D304.2 (A), IC301.5 (GND), IC301.6 (GND), IC301.7 (GND), IC301.8 (GND), IC302.2 (GND), R301.2, R302.1, R304.1, R306.1, X301.3, X302.0, X302.A1 (GND), X302.A12 (GND), X303.1 (GND), Y301.2 (GND), Y301.4 (GND)
- net V_EXT: no longer names the net of C301.1, D301.1 (K), X301.1
- net V_EXT: no longer IC301.1 (VIN)
- removed net V_USB: C305.2, D302.2 (A), X302.A4 (VBUS), X302.A9 (VBUS), X303.16 (VCC)
- new net: X302.A4 (VBUS), X302.A9 (VBUS)
- new net: D301.2 (A), X301.3
- new net: C305.2, X303.16 (VCC)
- new net: D302.1 (K), D303.1 (K), SW301.1
- new net: IC301.5 (GND), IC301.6 (GND), IC301.7 (GND), IC301.8 (GND)
- new net: SW301.2, SW301.3
- no-connect marks 0 -> 11
