File: pcb/sensors_interfaces.kicad_sch (KiCad schematic)
At the start: 25 parts, among them IC601 STK8321, IC602 SP3485EN-L_TR, IC603 WM8782SEDS_RV_C323842, IC604 CS4344-CZZ, IC605 MCP9700AT-E_TT, X601 KF2EDGR-3.81-3P, X602 PJ-327C-4A, X603 PJ-327C-4A

Commit message: make it work
Parts:
- removed IC601: STK8321, LGA-12_L2.0-W2.0-P0.50-TR, symbol eduboardv2:STK8321
- removed IC603: WM8782SEDS_RV_C323842, SSOP-20_L7.5-W5.2-P0.65-LS8.0-BL, symbol eduboardv2:WM8782SEDS_RV_C323842
- removed IC605: MCP9700AT-E_TT, SOT-23-3_L2.9-W1.3-P1.90-LS2.4-BR, symbol eduboardv2:MCP9700AT-E_TT
- removed X602: PJ-327C-4A, AUDIO-SMD_PJ-327C-4A, symbol eduboardv2:PJ-327C-4A
Connections:
- removed net +3.3V: C601.2, C602.2, IC602.8 (VCC), L601.1, R603.2
- removed net GND: C601.1, C602.1, C603.1, C604.1, C605.1, C608.1, C609.1, IC602.5 (GND), IC604.8 (GND), R601.1, R604.1, R605.1, X601.2, X603.1
- new net: C602.2, L601.1
- new net: C601.2, IC602.8 (VCC)
