File: pcb/up_rtc_flash.kicad_sch (KiCad schematic)
At the start: 13 parts, among them IC201 STK8321, IC202 PCF8563T_5,518, IC203 W25Q128JVSIQTR, X201 PCIE-52P40H, X202 32.768 kHz, X203 TF-15×15

Commit message: make it work
Parts:
- removed IC201: STK8321, LGA-12_L2.0-W2.0-P0.50-TR, symbol eduboardv2:STK8321
- removed X201: PCIE-52P40H, PCIE-SMD_PCIE-52P40H, symbol eduboardv2:PCIE-52P40H
Connections:
- net at C201.1, X202.2: now also IC202.1 (OSCI); no longer IC202.9 (OSCI)
- removed net +3.3V: C202.2, C204.2, D201.2 (+), IC203.8 (VCC), X203.4 (VDD)
- removed net GND: B201.2, C201.2, C202.1, C203.1, C204.1, IC202.4 (VSS), IC203.4 (GND), X203.6 (VSS)
- new net: C204.2, IC203.8 (VCC)
- new net: C202.2, X203.4 (VDD)
- no-connect marks 0 -> 9
