File: pcb/EduboardV2_Baseboard.kicad_pcb (KiCad board)
At the start: 2 copper layers, 144 parts, among them IC201 STK8321, IC202 PCF8563T_5,518, IC203 W25Q128JVSIQTR, IC301 XL1509-5.0E1, IC302 SY8113BADC, IC601 STK8321, IC602 SP3485EN-L_TR, IC603 WM8782SEDS_RV_C323842, IC604 CS4344-CZZ, IC605 MCP9700AT-E_TT, SW401 K2-1102SP-C4SC-04, SW402 K2-1102SP-C4SC-04, SW403 K2-1102SP-C4SC-04, SW404 K2-1102SP-C4SC-04, T401 AO3400A, T402 AO3400A, T403 AO3400A, T404 AO3400A, T405 AO3400A, X201 PCIE-52P40H, X202 32.768 kHz, X203 TF-15×15, X301 KF2EDGR-3.81-3P, X302 USB3.1C16PFSMT, X303 CH340G, X401 ER-TFT035-6, X501 PH-00650, X502 S4B-PH-SM4-K-TB(LF)(SN), X503 USB3.1C16PFSMT, X601 KF2EDGR-3.81-3P, X602 PJ-327C-4A, X603 PJ-327C-4A, Y301 X322512MSB4SI

Commit message: make it work
Parts:
- added SW301: 1FS1T1B9M2RES-5, eduboardv2:SW-TH_1FS1T1B9M2RES-5, F.Cu at (60.0, 37.0)
- X501: value PH-00650 -> BH-00105; footprint eduboardv2:HDR-SMD_40P-P2.54-V-M-R2-C20-S7.8-EH -> eduboardv2:IDC-SMD_BH-00105
- moved IC203 189.2 mm to (72.0, 93.0), turned to 180 degrees
- moved X203 173.8 mm to (64.1, 55.0), turned to 180 degrees
- moved X603 151.2 mm to (60.8, 98.0), turned to 90 degrees
- moved IC603 146.7 mm to (72.0, 82.0)
- moved D401 140.7 mm to (69.0, 165.0), turned to 90 degrees
- moved SW404 139.2 mm to (93.0, 174.0), turned to 180 degrees
- moved D404 138.9 mm to (93.0, 165.0), turned to 90 degrees
- moved X602 138.5 mm to (61.0, 87.0), turned to 90 degrees
- moved B201 132.2 mm to (86.0, 71.0), turned to -90 degrees
- moved D402 129.5 mm to (77.0, 165.0), turned to 90 degrees
- moved IC202 127.0 mm to (74.0, 62.0)
- moved SW401 121.8 mm to (85.0, 174.0), turned to 180 degrees
- moved D305 110.5 mm to (68.0, 42.0), turned to 90 degrees
- moved C201 107.9 mm to (179.8, 104.3)
- moved D201 107.9 mm to (174.2, 115.0)
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Connections:
- D302 pad 1: +5V -> Net-(D302-Pad1)
- D303 pad 1: +5V -> Net-(D302-Pad1)
- IC202 pad 1: (no net) -> Net-(C201-Pad1)
Routing:
- net (no net): vias 0 -> 4
Other:
- board outline added: 100 x 160 mm

Commit message: make it work 2
Parts:
- removed B201: CR2032-BS-6-1, eduboardv2:BAT-TH_CR2032-BS-6-1
- removed BUZZER401: MLT-8530, eduboardv2:BUZ-SMD_4P-L8.5-W8.5-P8.50-TL
- removed C201: 10pF, eduboardv2:C0402
- removed C202, C410, C411: 1uF, eduboardv2:C0402
- removed C203, C402, C404, C406, C408: 10nF, eduboardv2:C0402
- removed C204, C407, C409, C601, C602, C604: 100nF, eduboardv2:C0402
- removed C301, C309, C316: 220uF, 35V, eduboardv2:CAP-SMD_BD8.0-L8.3-W8.3-RD
- removed C302, C305, C306, C311, C314: 100nF, 50V, eduboardv2:C0402
- removed C303, C304, C308: 22pF, eduboardv2:C0402
- removed C307, C310, C313: 10uF, X5R, 25V, eduboardv2:C0603
- removed C312, C315: 1uF, 25V, eduboardv2:C0402
- removed C401, C403, C405: 1nF, eduboardv2:C0402
- removed C603, C605: 10uF, eduboardv2:C0603
- removed C606, C607: 4.7uF, eduboardv2:C0603
- removed C608, C609: 2.2nF, eduboardv2:C0402
- removed D201, D202: B5819W_C8598, eduboardv2:SOD-123_L2.7-W1.6-LS3.7-RD-1
- removed D301, D302, D303, D304: SS210, eduboardv2:SMA_L4.3-W2.6-LS5.2-RD
- removed D305, D401, D402, D403, D404, D405, D406, D407, D408: blue, eduboardv2:LED0603-R-RD_BLUE
- removed D409: RGB-LED, eduboardv2:LED-SMD_FM-B2020RGBA-HG
- removed D410: WS2812B-B_W, eduboardv2:LED-SMD_4P-L5.0-W5.0-TL_WS2812B-B
- removed D411: 1N4148WST4, eduboardv2:SOD-323_L1.8-W1.3-LS2.5-RD
- removed IC201, IC601: STK8321, eduboardv2:LGA-12_L2.0-W2.0-P0.50-TR
- removed IC202: PCF8563T_5,518, eduboardv2:SOIC-8_L5.0-W4.0-P1.27-LS6.0-BL
- removed IC203: W25Q128JVSIQTR, eduboardv2:SOIC-8_L5.3-W5.3-P1.27-LS8.0-BL
- removed IC301: XL1509-5.0E1, eduboardv2:SOIC-8_L5.0-W4.0-P1.27-LS6.0-BL
- removed IC302: SY8113BADC, eduboardv2:TSOT-23-6_L2.9-W1.6-P0.95-LS2.8-BR
- removed IC602: SP3485EN-L_TR, eduboardv2:SOIC-8_L5.0-W4.0-P1.27-LS6.0-BL
- removed IC603: WM8782SEDS_RV_C323842, eduboardv2:SSOP-20_L7.5-W5.2-P0.65-LS8.0-BL
- removed IC604: CS4344-CZZ, eduboardv2:TSSOP-10_L3.0-W3.0-P0.50-LS4.9-BL
- removed IC605: MCP9700AT-E_TT, eduboardv2:SOT-23-3_L2.9-W1.3-P1.90-LS2.4-BR
- removed L301: 6.8uH, 1A, eduboardv2:IND-SMD_L4.0-W4.0
- removed L302: 68uH, 1A, eduboardv2:IND-SMD_L6.0-W6.0_FNR60XXS
- removed L601: GZ1608D601TF, eduboardv2:L0603
- removed R301, R302: 5.1k, eduboardv2:R0402
- removed R303, R305: 100k, eduboardv2:R0402
- removed R304: 22k, eduboardv2:R0402
- removed R306, R401, R403, R405, R406, R407, R408, R410, R412, R413, R414, R416, R420: 1k, eduboardv2:R0402
- removed R402, R409, R417, R421, R601, R603, R604, R605: 10k, eduboardv2:R0402
- removed R404, R411, R415: 50k, eduboardv2:RES-TH_RK09K1130AAU
- removed R418, R419, R422: 150R, eduboardv2:R0402
- removed R423, R424, R425, R426, R427, R428, R430, R432, R433, R435: 10R, eduboardv2:R0402
- removed R429, R431, R434: NP, eduboardv2:R0402
- removed R602: 120R, eduboardv2:R0402
- removed R606, R607: 470R, eduboardv2:R0402
- removed SW301: 1FS1T1B9M2RES-5, eduboardv2:SW-TH_1FS1T1B9M2RES-5
- removed SW401, SW402, SW403, SW404: K2-1102SP-C4SC-04, eduboardv2:KEY-SMD_4P-L6.0-W6.0-P4.50-LS9.5-BL
- removed T401, T402, T403, T404, T405: AO3400A, eduboardv2:SOT-23-3_L2.9-W1.6-P1.90-LS2.8-BR
- removed X201: PCIE-52P40H, eduboardv2:PCIE-SMD_PCIE-52P40H
- removed X202: 32.768 kHz, eduboardv2:FC-135R_L3.2-W1.5
- removed X203: TF-15×15, eduboardv2:TF-SMD_TF-15-15
- removed X301, X601: KF2EDGR-3.81-3P, eduboardv2:CONN-TH_3P-P3.81_KF2EDGR-3.81-3P
- removed X302, X503: USB3.1C16PFSMT, eduboardv2:USB-C-SMD_TYPE-C-USB-17
- removed X303: CH340G, eduboardv2:SOIC-16_L9.9-W3.9-P1.27-LS6.0-BL
- removed X401: ER-TFT035-6, eduboardv2:FPC-SMD_AFC07-S50ECA-00
- removed X501: BH-00105, eduboardv2:IDC-SMD_BH-00105
- removed X502: S4B-PH-SM4-K-TB(LF)(SN), eduboardv2:CONN-SMD_S4B-PH-SM4-K-TB-LF-SN
- removed X602, X603: PJ-327C-4A, eduboardv2:AUDIO-SMD_PJ-327C-4A
- removed Y301: X322512MSB4SI, eduboardv2:OSC-SMD_4P-L3.2-W2.5-BL
